File: schematics/LED-board.brd (EAGLE design)
At the start: 100 x 80 mm, 7 parts

Commit message: Reworked some schematics
Parts:
- added U$1: (no value), bfl:OSHW2
- moved LED2 40.7 mm to (10.0, 37.0)
- moved SV1 34.5 mm to (9.68, 4.40)
- moved LED1 34.2 mm to (10.0, 17.0)
- moved R1 33.3 mm to (7.95, 11.0), flipped to the bottom, turned to 180 degrees
- moved R3 29.0 mm to (8.05, 51.0), flipped to the bottom, turned to 180 degrees
- moved R2 27.4 mm to (7.95, 31.0), flipped to the bottom, turned to 180 degrees
- moved LED3 3.31 mm to (10.0, 57.0)
Connections:
- net N$7 renamed GND
Routing:
- net N$6: track 0.00 -> 51.3 mm
- net N$5: track 0.00 -> 31.8 mm
- net N$4: track 0.00 -> 11.6 mm
- net N$3: track 0.00 -> 8.48 mm
- net N$2: track 0.00 -> 8.42 mm
- net N$1: track 0.00 -> 8.42 mm
- added copper zone on layer 16, net GND
Other:
- board size 100 x 80 mm -> 20 x 67 mm
- board text added: "OSS spectro v0.3"
