File: schematics/LED-board.sch (EAGLE design)
At the start: 7 parts

Commit message: Reworked some schematics
Connections:
- net N$7 renamed GND
Changed lines of the file:
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@@
 </segment>
 </net>
-<net name="N$7" class="0">
+<net name="GND" class="0">
 <segment>
 <pinref part="LED1" gate="G$1" pin="C"/>
