File: schematics/Controller-Bee/Controller-Bee.sch (KiCad schematic (older format))
At the start: 20 parts, among them P1 CONN_01X05, P2 CONN_02X04, P3 USB_OTG, P4 CONN_02X04, U1 EFM8UB10F8G-B-QFN20

Commit message: schematics: update LED connections, use 4x resistor arrays
Connections:
- net VDD: no longer P4.3 (P3), P4.5 (P5), P4.7 (P7), P4.8 (P8)
- no-connect marks 4 -> 8
Changed lines of the file:
@@
 LIBS:contrib
 LIBS:valves
-LIBS:efm8ub10f8g-b-qfn20
 LIBS:Controller-Bee-cache
 EELAYER 25 0
@@
 	1    0    0    -1
 $EndComp
-Wire Wire Line
-	10450 4850 10450 5600
-Wire Wire Line
-	10450 5000 10300 5000
-Wire Wire Line
-	10450 5600 9650 5600
-Wire Wire Line
-	9650 5600 9650 5300
-Wire Wire Line
-	9650 5300 9800 5300
-Connection ~ 10450 5000
-Wire Wire Line
-	10300 5100 10450 5100
-Connection ~ 10450 5100
-Wire Wire Line
-	10300 5200 10450 5200
-Connection ~ 10450 5200
-Wire Wire Line
-	10300 5300 10450 5300
-Connection ~ 10450 5300
 $Comp
 L GND #PWR08
@@
 Text Label 4650 3800 0    60   ~ 0
 d-
+Wire Wire Line
+	10300 5000 10450 5000
+Wire Wire Line
+	10450 5000 10450 4850
+NoConn ~ 10300 5100
+NoConn ~ 10300 5200
+NoConn ~ 10300 5300
+NoConn ~ 9800 5300
 $EndSCHEMATC
