File: schematics/Controller-Nano-i2c_mux/Controller-Nano-i2c_mux-Square.kicad_pcb (KiCad board)
At the start: 2 copper layers, 50 x 50 mm, 28 parts, among them P1 CONN_02X04, P2 CONN_02X04, P3 CONN_01X04, P4 CONN_01X04, U1 Arduino_Nano, U2 PCA9544A

Commit message: schematics: update LED connections, use 4x resistor arrays
Parts:
- removed R1, R3, R5: 330, Resistors_SMD:R_0805
- removed R2, R4, R6: 470, Resistors_SMD:R_0805
- removed the REF** at (130.0, 76.0)
- removed the REF** at (130.0, 118.0)
- removed the REF** at (172.0, 118.0)
- removed the REF** at (172.0, 76.0)
- added P5: CONN_01X01, Connect:1pin, F.Cu at (172.0, 117.0)
- added P6: CONN_01X01, Connect:1pin, F.Cu at (130.0, 117.0)
- added P7: CONN_01X01, Connect:1pin, F.Cu at (130.0, 77.0)
- added P8: CONN_01X01, Connect:1pin, F.Cu at (172.0, 77.0)
- added RP2: R_PACK4, Resistors_SMD:R_Array_Convex_4x0603, B.Cu at (145.9, 75.5)
- R10, R11: value R -> 4k7
- R7, R8, R9: value R -> 220
- REF**: value Symbol_OSHW-Logo_CopperTop -> Symbol_OSHW-Logo_SilkScreen
- RP1: value R_PACK8 -> R_PACK4; footprint Resistors_SMD:R_Array_Convex_8x0602 -> Resistors_SMD:R_Array_Convex_4x0603
- moved RP1 2.16 mm to (152.9, 75.5)
- moved REF** 1.04 mm to (130.3, 107.0)
Connections:
- P2 pad 3: +3V3 -> (no net)
- P2 pad 5: +3V3 -> (no net)
- P2 pad 7: +3V3 -> (no net)
- P2 pad 8: +3V3 -> (no net)
- R7 pad 2: Net-(R7-Pad2) -> LED1
- R8 pad 2: Net-(R8-Pad2) -> LED2
- R9 pad 2: Net-(R9-Pad2) -> LED3
- RP1 pad 5: SC2 -> +3V3
- RP1 pad 6: SC1 -> +3V3
- RP1 pad 7: SC0 -> +3V3
- RP1 pad 8: SDA -> +3V3
- U1 pad 1: Net-(U1-Pad1) -> (no net)
- U1 pad 10: Net-(R6-Pad1) -> (no net)
- U1 pad 18: Net-(U1-Pad18) -> (no net)
- U1 pad 19: Net-(U1-Pad19) -> (no net)
- U1 pad 2: Net-(U1-Pad2) -> (no net)
- U1 pad 20: Net-(R9-Pad2) -> (no net)
- U1 pad 21: Net-(R8-Pad2) -> (no net)
- U1 pad 22: Net-(R7-Pad2) -> (no net)
- U1 pad 25: Net-(U1-Pad25) -> (no net)
- U1 pad 26: Net-(U1-Pad26) -> (no net)
- U1 pad 27: Net-(U1-Pad27) -> (no net)
- U1 pad 28: Net-(U1-Pad28) -> (no net)
- U1 pad 29: Net-(U1-Pad29) -> (no net)
- U1 pad 3: Net-(U1-Pad3) -> (no net)
- U1 pad 30: Net-(U1-Pad30) -> (no net)
- U1 pad 5: Net-(R1-Pad1) -> LED1
- U1 pad 6: Net-(R2-Pad1) -> (no net)
- U1 pad 7: Net-(R3-Pad1) -> LED2
- U1 pad 8: Net-(R4-Pad1) -> (no net)
- U1 pad 9: Net-(R5-Pad1) -> LED3
- U2 pad 11: Net-(U2-Pad11) -> (no net)
- U2 pad 14: Net-(U2-Pad14) -> (no net)
- U2 pad 15: Net-(U2-Pad15) -> (no net)
- U2 pad 16: Net-(U2-Pad16) -> (no net)
- U2 pad 17: Net-(U2-Pad17) -> (no net)
- U2 pad 4: Net-(U2-Pad4) -> (no net)
- U2 pad 7: Net-(U2-Pad7) -> (no net)
Routing:
- net LED2: track 36.9 -> 78.2 mm
- net LED3: track 27.4 -> 65.2 mm
- net Net-(R7-Pad2): track 37.4 -> 0.00 mm, vias 1 -> 0
- net Net-(R8-Pad2): track 30.9 -> 0.00 mm
- net LED1: track 53.6 -> 77.0 mm
- net Net-(R9-Pad2): track 18.5 -> 0.00 mm
- net Net-(R6-Pad1): track 14.3 -> 0.00 mm
- net Net-(R5-Pad1): track 12.1 -> 0.00 mm
- net Net-(R1-Pad1): track 8.79 -> 0.00 mm
- net Net-(R4-Pad1): track 8.27 -> 0.00 mm
- net SC1: track 29.7 -> 36.6 mm
- net +3V3: track 188.1 -> 195.1 mm, vias 3 -> 4
- net Net-(R2-Pad1): track 6.91 -> 0.00 mm
- net Net-(R3-Pad1): track 6.84 -> 0.00 mm
- net SC0: track 30.3 -> 36.8 mm
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Other:
- net class Power: trace_width 0.25 -> 1
- board text added: "1"

Commit message: Schematics update
Other:
- board text added: "DIλ Controller board v0.9-Nano-s"
- board text removed: "DIλ Controller Board v0.9-Nano-s"
Changed lines of the file:
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@@
 (kicad_pcb (version 4) (host pcbnew "(2015-08-06 BZR 6060)-product")
   (general
-    (links 0)
-    (no_connects 19)
-    (area 125.924999 71.924999 176.075001 122.075001)
+    (links 70)
+    (no_connects 0)
+    (area 122 65.798699 180.000001 127.858501)
     (thickness 1.6)
     (drawings 14)
@@
     (visible_elements FFFFFF7F)
     (pcbplotparams
-      (layerselection 0x00030_80000001)
-      (usegerberextensions false)
+      (layerselection 0x010f0_80000001)
+      (usegerberextensions true)
       (excludeedgelayer true)
       (linewidth 0.100000)
@@
       (viasonmask false)
       (mode 1)
-      (useauxorigin false)
+      (useauxorigin true)
       (hpglpennumber 1)
       (hpglpenspeed 20)
@@
       (plotvalue true)
       (plotinvisibletext false)
-      (padsonsilk false)
+      (padsonsilk true)
       (subtractmaskfromsilk false)
       (outputformat 1)
       (mirror false)
-      (drillshape 1)
+      (drillshape 0)
       (scaleselection 1)
-      (outputdirectory ""))
+      (outputdirectory Controller-Nano-i2c_mux-Square/))
   )
   (net 0 "")
@@
     (effects (font (size 1.5 1.5) (thickness 0.3)))
   )
-  (gr_text "DIλ\nController Board\nv0.9-Nano-s\n\n" (at 132 92 90) (layer F.SilkS)
+  (gr_text "DIλ\nController board\nv0.9-Nano-s\n\n" (at 132 92 90) (layer F.SilkS)
     (effects (font (size 1.5 1.5) (thickness 0.3) italic))
   )
