File: schematics/Controller-Nano-i2c_mux/Controller-Nano-i2c_mux.sch (KiCad schematic (older format))
At the start: 23 parts, among them P1 CONN_02X04, P2 CONN_02X04, P3 CONN_01X04, P4 CONN_01X04, U1 Arduino_Nano, U2 PCA9544A

Commit message: schematics: update LED connections, use 4x resistor arrays
Parts:
- removed R1, R3, R5: 330, Resistors_SMD:R_0805, symbol R
- removed R2, R4, R6: 470, Resistors_SMD:R_0805, symbol R
- removed RP1: R_PACK8, Resistors_SMD:R_Array_Convex_8x0602, symbol R_PACK8
- added P5, P6, P7, P8: CONN_01X01, Connect:1pin, symbol CONN_01X01
- added RP1, RP2: R_PACK4, Resistors_SMD:R_Array_Convex_4x0603, symbol R_PACK4
- renumbered D3 to LED1, D2 to LED2, D1 to LED3
Connections:
- net +3V3: now also RP1.5 (R4), RP1.6 (R3), RP1.7 (R2), RP1.8 (R1), RP2.5 (R4), RP2.6 (R3), RP2.7 (R2), RP2.8 (R1); no longer P2.3 (P3), P2.5 (P5), P2.7 (P7), P2.8 (P8)
- net GND: now also P5.1 (P1), P6.1 (P1), P7.1 (P1), P8.1 (P1)
- net LED1: now also R7.2, U1.5 (D2)
- net LED2: now also R8.2, U1.7 (D4)
- net LED3: now also R9.2, U1.9 (D6)
- net SC0: now also RP2.3 (P3)
- net SC1: now also RP2.2 (P2)
- net SC2: now also RP2.1 (P1)
- net SCL: now also RP1.1 (P1)
- net SD0: now also RP1.2 (P2)
- net SD1: now also RP1.3 (P3)
- net SD2: now also RP1.4 (P4)
- net SDA: now also RP2.4 (P4)
- net at U1.20 (A1): no longer R9.2
- net at U1.21 (A2): no longer R8.2
- net at U1.22 (A3): no longer R7.2
- no-connect marks 18 -> 22

Commit message: Schematics update
Other:
- note added: "I2C multiplexer"
- note added: "Metalized through holes\n(optional)"
- note added: "Optional legacy interface.\n"
- note removed: "Optional stuff to connect to older LED/Sensor boards\n"
- moved on the sheet: C1, C2, LED1, LED2, LED3, P1, P2, P3, P4, P5, P6, P7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
