File: schematics/Sensor-Board-LTR329-3x/Sensor-Board-LTR329-3x-1cm.kicad_pcb (KiCad board)
At the start: 2 copper layers, 10 x 48 mm, 10 parts, among them P1 CONN_02X04, U1 LTR-329ALS-01, U2 LTR-329ALS-01, U3 LTR-329ALS-01

Commit message: Schematics update
Other:
- board text added: "1"
- board text added: "DIλ Sensor Board v0.9-LTR329-3x-1cm"
- board text removed: "DIλ Sensor Board v0.9-LTR329-1cm"
Changed lines of the file:
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@@
-(kicad_pcb (version 4) (host pcbnew "(2015-08-06 BZR 6060)-product")
+(kicad_pcb (version 4) (host pcbnew "(2016-01-25 BZR 6514, Git a23e712)-product")
   (general
     (links 24)
     (no_connects 0)
-    (area 159.924999 61.924999 170.075001 110.075001)
+    (area 157.25 60.75 172.500001 111.250001)
     (thickness 1.6)
-    (drawings 7)
+    (drawings 8)
     (tracks 84)
     (zones 0)
@@
   (page A4)
   (layers
-    (0 F.Cu signal hide)
+    (0 F.Cu signal)
     (31 B.Cu signal)
     (32 B.Adhes user)
@@
     (pad_drill 0.762)
     (pad_to_mask_clearance 0.2)
-    (aux_axis_origin 0 0)
+    (aux_axis_origin 160 110)
     (visible_elements FFFFFF7F)
     (pcbplotparams
-      (layerselection 0x00030_80000001)
-      (usegerberextensions false)
+      (layerselection 0x010f0_80000001)
+      (usegerberextensions true)
       (excludeedgelayer true)
       (linewidth 0.100000)
@@
       (viasonmask false)
       (mode 1)
-      (useauxorigin false)
+      (useauxorigin true)
       (hpglpennumber 1)
       (hpglpenspeed 20)
@@
       (plotvalue true)
       (plotinvisibletext false)
-      (padsonsilk false)
+      (padsonsilk true)
       (subtractmaskfromsilk false)
       (outputformat 1)
       (mirror false)
-      (drillshape 1)
+      (drillshape 0)
       (scaleselection 1)
-      (outputdirectory ""))
+      (outputdirectory Sensor-Board-LTR329-3x-1cm/))
   )
   (net 0 "")
@@
     (descr "Pin Header 2mm 4x2pin")
     (tags "CONN DEV")
-    (fp_text reference P1 (at 0 5) (layer B.SilkS) hide
+    (fp_text reference P1 (at 0 3.5) (layer B.SilkS)
       (effects (font (size 1 1) (thickness 0.15)) (justify mirror))
     )
@@
       (net 8 SC2))
   )
-  (gr_text "DIλ Sensor Board\nv0.9-LTR329-1cm" (at 165.5 77.5 270) (layer B.SilkS)
+  (gr_text 1 (at 162 90.75 270) (layer B.SilkS)
     (effects (font (size 1.5 1.5) (thickness 0.3)) (justify mirror))
   )
+  (gr_text "DIλ Sensor Board\nv0.9-LTR329-3x-1cm" (at 165.5 77.5 270) (layer B.SilkS)
+    (effects (font (size 1.5 1.5) (thickness 0.3)) (justify mirror))
+  )
