File: schematics/Sensor-Board-TSL2561-3x/Sensor-Board-TSL2561-3x-1cm.kicad_pcb (KiCad board)
At the start: 2 copper layers, 10 x 48 mm, 10 parts, among them P1 CONN_02X04, U1 TSL2561, U2 TSL2561, U3 TSL2561

Commit message: Schematics update
Parts:
- P1: value CONN_02X04 -> eCONN_02X04
Other:
- board text added: "1"
